File: hardware/esp32-emon/esp32-emon.kicad_pcb (KiCad board)
At the start: 2 copper layers, 49.8 x 55.8 mm, 13 parts, among them J1 SJ-3523-SMT-TR, J2 Barrel_Jack, U1 ESP32-DEVKIT-V1

Commit message: Update from 1K to 10K
Parts:
- R5: value 1K -> 10K
Changed lines of the file:
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@@
         (effects (font (size 1 1) (thickness 0.15)))
     )
-    (fp_text value "1K" (at 3.81 -1.8 90) (layer "F.Fab")
+    (fp_text value "10K" (at 3.81 -1.8 90) (layer "F.Fab")
         (effects (font (size 1 1) (thickness 0.15)))
     )

Commit message: Test TurboCase
Parts:
- added ?: , TurboCase:Cutout_Pinheader_01x04_254, F.Cu at (140.8, 34.0)
- added REF**: MountingHole_3mm, MountingHole:MountingHole_3mm, F.Cu at (162.2, 30.1)
- added REF**: MountingHole_3mm, MountingHole:MountingHole_3mm, F.Cu at (186.7, 30.1)
- added REF**: MountingHole_3mm, MountingHole:MountingHole_3mm, F.Cu at (162.2, 77.1)
- added REF**: MountingHole_3mm, MountingHole:MountingHole_3mm, F.Cu at (186.7, 77.1)
